Commit message: Included libgazebo_ros_camera.so

File: urdf/simple_robot_nav2.urdf.xacro (robot description, xacro)
@@ -100,4 +100,18 @@
     </inertial>
   </link>
+<!-- libgazebo_ros_camera Link - forward facing camera -->
+  <link name="camera_point_link">
+    <collision>
+      <origin xyz="0 0 0.3" rpy="0 0 0"/>
+      <geometry>
+    <box size="0.1 0.1 0.1"/>
+      </geometry>
+    </collision>
+    <inertial>
+      <mass value="1e-5" />
+      <origin xyz="0 0 0" rpy="0 0 0"/>
+      <inertia ixx="1e-6" ixy="0" ixz="0" iyy="1e-6" iyz="0" izz="1e-6" />
+    </inertial>
+  </link>
 <!-- END of Link declaration -->
 <!-- Start of Joints - connecting all links together -->
@@ -142,4 +156,11 @@
         <limit effort="30" velocity="2.0" />
         <safety_controller k_velocity="10" k_position="15" soft_lower_limit="-2.0" soft_upper_limit="0.5" />
+    </joint>
+        <joint name="camera_joint" type="fixed">
+        <axis xyz="0 1 0" />
+        <origin xyz="-0.1 0 .4" rpy="0 0 ${PI}"/>
+        <parent link="base_link"/>
+        <child link="camera_point_link"/>
+            <dynamics damping="0.7"/>
     </joint>
     <joint name="hokuyo_joint" type="fixed">
@@ -220,4 +241,49 @@
         <slip2>1.000000</slip2>
   </gazebo>
+  <gazebo reference="camera_point_link">
+    <sensor type="camera" name="camera1">
+      <update_rate>30.0</update_rate>
+      <camera name="head">
+        <pose>0 0 0 0 0 0</pose>
+        <horizontal_fov>1.3962634</horizontal_fov>
+        <image>
+          <width>800</width>
+          <height>800</height>
+          <format>R8G8B8</format>
+        </image>
+        <clip>
+          <near>0.02</near>
+          <far>300</far>
+        </clip>
+        <noise>
+	  <type>gaussian</type>
+	  <!-- Noise is sampled independently per pixel on each frame.
+	  That pixel’s noise value is added to each of its color
+	  channels, which at that point lie in the range [0,1]. -->
+	  <mean>0.0</mean>
+	  <stddev>0.007</stddev>
+	</noise>
+      </camera>
+      <plugin name="camera_controller" filename="libgazebo_ros_camera.so">
+      <ros>
+        <!--namespace>custom_ns</namespace-->
+        <remapping>image_raw:=custom_img</remapping>
+        <!--remapping>camera_info:=custom_info</remapping-->
+      </ros>
+        <alwaysOn>true</alwaysOn>
+        <updateRate>0.0</updateRate>
+        <cameraName>camera</cameraName>
+        <imageTopicName>image_raw</imageTopicName>
+        <cameraInfoTopicName>camera_info</cameraInfoTopicName>
+        <frameName>camera_point_link</frameName>
+        <hackBaseline>0.07</hackBaseline>
+        <distortionK1>0.0</distortionK1>
+        <distortionK2>0.0</distortionK2>
+        <distortionK3>0.0</distortionK3>
+        <distortionT1>0.0</distortionT1>
+        <distortionT2>0.0</distortionT2>
+      </plugin>
+    </sensor>
+  </gazebo>
   <gazebo reference="hokuyo_link">
     <sensor name="lidar" type="ray">

Commit message: Edited libgazebo_ros_camera

File: urdf/simple_robot_nav2.urdf.xacro (robot description, xacro)
@@ -159,5 +159,5 @@
         <joint name="camera_joint" type="fixed">
         <axis xyz="0 1 0" />
-        <origin xyz="-0.1 0 .4" rpy="0 0 ${PI}"/>
+        <origin xyz="-0.1 0 .4" rpy="0 0 0"/>
         <parent link="base_link"/>
         <child link="camera_point_link"/>
