Commit message: update

File: urdf/KANE_mobile_robotics_hschoon.xacro (robot description, xacro)
@@ -18,13 +18,11 @@
         <collision name="chassis">
             <geometry>
-                <box size="0.5 0.278 0.245" /> <!-- HERE: "0.5 0.278 0.245" -->
+                <box size=".4 .2 .1" />
             </geometry>
         </collision>
         <visual name="chassis">
             <geometry>
-                <mesh filename="$(find mobile_robotics_hschoon)/meshes/chassis_v2.stl" scale="1.5 1.5 1.5" />
-            </geometry>
-            <origin xyz="0.0 0.0 0.05" rpy="0 0 3.14159"/>
-            <!-- <material name="Grey" /> -->
+                <box size=".4 .2 .1" />
+            </geometry>
         </visual>
     </link>
@@ -37,10 +35,10 @@
         <collision name="castor">
             <geometry>
-                <sphere radius=".043" /> <!-- HERE: ".04275" -->
+                <sphere radius=".05" />
             </geometry>
         </collision>
         <visual name="castor">
             <geometry>
-                <sphere radius=".043" />
+                <sphere radius=".05" />
             </geometry>
         </visual>
@@ -52,14 +50,13 @@
             <inertia ixx="0.004" ixy="0.0" ixz="0.0" iyy="0.004" iyz="0.0" izz="0.002"/>
         </inertial>
+        <pose>0.1 0.13 0.1 0 1.5707 1.5707</pose>
         <collision name="left_wheel">
             <geometry>
-                <!-- <mesh filename="$(find mobile_robotics_hschoon)/meshes/wheel.stl" scale="1.5 1.5 1.5" /> -->
-                <cylinder length="0.04" radius="0.043"/>
+                <cylinder radius='.1' length='.05'/>
             </geometry>
         </collision>
         <visual name="left_wheel">
             <geometry>
-                <!-- <mesh filename="$(find mobile_robotics_hschoon)/meshes/wheel.stl" scale="1.5 1.5 1.5" /> -->
-                <cylinder length="0.04" radius="0.043"/>
+                <cylinder radius='.1' length='.05'/>
             </geometry>
         </visual>
@@ -71,14 +68,13 @@
             <inertia ixx="0.004" ixy="0.0" ixz="0.0" iyy="0.004" iyz="0.0" izz="0.002"/>
         </inertial>
+        <pose>0.1 0.13 0.1 0 1.5707 1.5707</pose>
         <collision name="right_wheel">
             <geometry>
-                <!-- <mesh filename="$(find mobile_robotics_hschoon)/meshes/wheel.stl" scale="1.5 1.5 1.5" /> -->
-                <cylinder length="0.04" radius="0.043"/>
+                <cylinder radius='.1' length='.05'/>
             </geometry>
         </collision>
         <visual name="right_wheel">
             <geometry>
-                <!-- <mesh filename="$(find mobile_robotics_hschoon)/meshes/wheel.stl" scale="1.5 1.5 1.5" /> -->
-                <cylinder length="0.04" radius="0.043"/>
+                <cylinder radius='.1' length='.05'/>
             </geometry>
         </visual>
@@ -137,5 +133,5 @@
         <parent link="chassis"/>
         <child link="castor"/>
-        <origin xyz=".125 0 -0.14" rpy="0 0 0"/>
+        <origin xyz=".15 0 -.05" rpy="0 0 0"/>
         <axis xyz="0 1 0"/>
         <dynamics damping="0.7"/>
@@ -144,6 +140,6 @@
         <parent link="chassis"/>
         <child link="left_wheel"/>
-        <origin xyz="-0.187 0.0834 -0.14" rpy="0 1.5707 1.5707"/> <!-- HERE: "0 1.5707 0" -->
-        <axis xyz="0 0 1"/> <!-- HERE: ""0 1 0" -->
+        <origin xyz="-0.1 0.13 0" rpy="0 1.5707 1.5707"/>
+        <axis xyz="0 0 1"/>
         <calibration rising="0.0"/>
         <dynamics damping="0.0" friction="0.0"/>
@@ -154,6 +150,6 @@
         <parent link="chassis"/>
         <child link="right_wheel"/>
-        <origin xyz="-0.187 -0.0834 -0.14" rpy="0 1.5707 1.5707"/> <!-- HERE: "-3.14159 -1.5707 0" -->
-        <axis xyz="0 0 1"/>  <!-- HERE: ""0 -1 0" -->
+        <origin xyz="-0.1 -0.13 0" rpy="0 1.5707 1.5707"/>
+        <axis xyz="0 0 1"/>
         <calibration rising="0.0"/>
         <dynamics damping="0.0" friction="0.0"/>
@@ -161,5 +157,5 @@
         <safety_controller k_velocity="10" k_position="15" soft_lower_limit="-2.0" soft_upper_limit="0.5" />
     </joint>
-        <joint name="camera_joint" type="fixed">
+    <joint name="camera_joint" type="fixed">
         <axis xyz="0 1 0" />
         <origin xyz="-0.1 0 .2" rpy="0 0 0"/>
@@ -217,5 +213,5 @@
     	<mu1>.01</mu1>
     	<mu2>.01</mu2>
-        <fdir1>0.000000 0.000000 0.000000</fdir1>
+        <fdir1>1.000000 0.000000 0.000000</fdir1>
         <slip1>1.000000</slip1>
         <slip2>1.000000</slip2>
@@ -225,5 +221,5 @@
     	<mu1>100000</mu1>
     	<mu2>100000</mu2>
-        <fdir1>0.000000 0.000000 0.000000</fdir1>
+        <fdir1>1.000000 0.000000 0.000000</fdir1>
         <slip1>0.000000</slip1>
         <slip2>0.000000</slip2>
@@ -233,5 +229,5 @@
     	<mu1>100000</mu1>
     	<mu2>100000</mu2>
-        <fdir1>0.000000 0.000000 0.000000</fdir1>
+        <fdir1>1.000000 0.000000 0.000000</fdir1>
         <slip1>0.000000</slip1>
         <slip2>0.000000</slip2>
@@ -241,5 +237,5 @@
     	<mu1>.01</mu1>
     	<mu2>.01</mu2>
-        <fdir1>0.000000 0.000000 0.000000</fdir1>
+        <fdir1>1.000000 0.000000 0.000000</fdir1>
         <slip1>1.000000</slip1>
         <slip2>1.000000</slip2>
@@ -307,5 +303,5 @@
         <range>
           <min>0.120000</min>
-          <max>8.0</max>
+          <max>13.5</max>
           <resolution>0.015000</resolution>
         </range>
