Commit message: update 20230703 - marker debugging started

File: urdf/mobile_robotics_hschoon.xacro (robot description, xacro)
@@ -18,5 +18,5 @@
         <collision name="chassis">
             <geometry>
-                <box size="0.5 0.278 0.245" />
+                <box size="0.5 0.278 0.245" /> <!-- HERE: "0.5 0.278 0.245" -->
             </geometry>
         </collision>
@@ -26,5 +26,5 @@
             </geometry>
             <origin xyz="0.0 0.0 0.05" rpy="0 0 3.14159"/>
-            <material name="Grey" />
+            <!-- <material name="Grey" /> -->
         </visual>
     </link>
@@ -37,5 +37,5 @@
         <collision name="castor">
             <geometry>
-                <sphere radius=".04275" />
+                <sphere radius=".043" /> <!-- HERE: ".04275" -->
             </geometry>
         </collision>
@@ -54,10 +54,12 @@
         <collision name="left_wheel">
             <geometry>
-                <mesh filename="$(find mobile_robotics_hschoon)/meshes/wheel.stl" scale="1.5 1.5 1.5" />
+                <!-- <mesh filename="$(find mobile_robotics_hschoon)/meshes/wheel.stl" scale="1.5 1.5 1.5" /> -->
+                <cylinder length="0.04" radius="0.043"/>
             </geometry>
         </collision>
         <visual name="left_wheel">
             <geometry>
-                <mesh filename="$(find mobile_robotics_hschoon)/meshes/wheel.stl" scale="1.5 1.5 1.5" />
+                <!-- <mesh filename="$(find mobile_robotics_hschoon)/meshes/wheel.stl" scale="1.5 1.5 1.5" /> -->
+                <cylinder length="0.04" radius="0.043"/>
             </geometry>
         </visual>
@@ -71,10 +73,12 @@
         <collision name="right_wheel">
             <geometry>
-                <mesh filename="$(find mobile_robotics_hschoon)/meshes/wheel.stl" scale="1.5 1.5 1.5" />
+                <!-- <mesh filename="$(find mobile_robotics_hschoon)/meshes/wheel.stl" scale="1.5 1.5 1.5" /> -->
+                <cylinder length="0.04" radius="0.043"/>
             </geometry>
         </collision>
         <visual name="right_wheel">
             <geometry>
-                <mesh filename="$(find mobile_robotics_hschoon)/meshes/wheel.stl" scale="1.5 1.5 1.5" />
+                <!-- <mesh filename="$(find mobile_robotics_hschoon)/meshes/wheel.stl" scale="1.5 1.5 1.5" /> -->
+                <cylinder length="0.04" radius="0.043"/>
             </geometry>
         </visual>
@@ -140,6 +144,6 @@
         <parent link="chassis"/>
         <child link="left_wheel"/>
-        <origin xyz="-0.167 0.0834 -0.14" rpy="0 1.5707 0"/>
-        <axis xyz="0 1 0"/>
+        <origin xyz="-0.187 0.0834 -0.14" rpy="0 1.5707 1.5707"/> <!-- HERE: "0 1.5707 0" -->
+        <axis xyz="0 0 1"/> <!-- HERE: ""0 1 0" -->
         <calibration rising="0.0"/>
         <dynamics damping="0.0" friction="0.0"/>
@@ -150,6 +154,6 @@
         <parent link="chassis"/>
         <child link="right_wheel"/>
-        <origin xyz="-0.167 -0.0834 -0.14" rpy="-3.14159 -1.5707 0"/>
-        <axis xyz="0 -1 0"/>
+        <origin xyz="-0.187 -0.0834 -0.14" rpy="0 1.5707 1.5707"/> <!-- HERE: "-3.14159 -1.5707 0" -->
+        <axis xyz="0 0 1"/>  <!-- HERE: ""0 -1 0" -->
         <calibration rising="0.0"/>
         <dynamics damping="0.0" friction="0.0"/>
@@ -159,5 +163,5 @@
         <joint name="camera_joint" type="fixed">
         <axis xyz="0 1 0" />
-        <origin xyz="-0.1 0 .4" rpy="0 0 0"/>
+        <origin xyz="-0.1 0 .2" rpy="0 0 0"/>
         <parent link="base_link"/>
         <child link="camera_point_link"/>
@@ -166,5 +170,5 @@
     <joint name="hokuyo_joint" type="fixed">
         <axis xyz="0 1 0" />
-        <origin xyz="-0.1 0 .14" rpy="0 0 3.1415926535897931"/>
+        <origin xyz="-0.1 0 .15" rpy="0 0 3.1415926535897931"/> <!-- HERE: "-0.1 0 .14" -->
         <parent link="base_link"/>
         <child link="hokuyo_link"/>
@@ -221,5 +225,5 @@
     	<mu1>100000</mu1>
     	<mu2>100000</mu2>
-        <fdir1>0.000000 0.000000 0.000000</fdir1>
+        <fdir1>1.000000 0.000000 0.000000</fdir1>
         <slip1>0.000000</slip1>
         <slip2>0.000000</slip2>
@@ -229,5 +233,5 @@
     	<mu1>100000</mu1>
     	<mu2>100000</mu2>
-        <fdir1>0.000000 0.000000 0.000000</fdir1>
+        <fdir1>1.000000 0.000000 0.000000</fdir1>
         <slip1>0.000000</slip1>
         <slip2>0.000000</slip2>
@@ -237,5 +241,5 @@
     	<mu1>.01</mu1>
     	<mu2>.01</mu2>
-        <fdir1>0.000000 0.000000 0.000000</fdir1>
+        <fdir1>1.000000 0.000000 0.000000</fdir1>
         <slip1>1.000000</slip1>
         <slip2>1.000000</slip2>
@@ -303,5 +307,5 @@
         <range>
           <min>0.120000</min>
-          <max>3.5</max>
+          <max>13.5</max>
           <resolution>0.015000</resolution>
         </range>

Commit message: update

File: urdf/mobile_robotics_hschoon.xacro (robot description, xacro)
@@ -4,4 +4,7 @@
   <material name="Grey">
     <color rgba="0.7 0.7 0.7 1.0"/>
+  </material>
+  <material name="barbiepink" >
+    <color rgba="0.996078431372549 0.27450980392156865 0.6470588235294118 1.0" />
   </material>
 <!-- Start of Links - first link must be a non-inertial link -->
@@ -23,8 +26,7 @@
         <visual name="chassis">
             <geometry>
-                <mesh filename="$(find mobile_robotics_hschoon)/meshes/chassis_v2.stl" scale="1.5 1.5 1.5" />
+                <mesh filename="$(find mobile_robotics_hschoon)/meshes/chassis.dae" scale="1.5 1.5 1.5" />
             </geometry>
             <origin xyz="0.0 0.0 0.05" rpy="0 0 3.14159"/>
-            <!-- <material name="Grey" /> -->
         </visual>
     </link>
@@ -37,5 +39,5 @@
         <collision name="castor">
             <geometry>
-                <sphere radius=".043" /> <!-- HERE: ".04275" -->
+                <sphere radius=".043" />
             </geometry>
         </collision>
@@ -107,7 +109,7 @@
   <link name="camera_point_link">
     <collision>
-      <origin xyz="0 0 0.3" rpy="0 0 0"/>
+      <origin xyz="0 0.2 0.3" rpy="0 0 0"/>
       <geometry>
-    <box size="0.1 0.1 0.1"/>
+         <box size="0.1 0.1 0.1"/>
       </geometry>
     </collision>
@@ -163,5 +165,5 @@
         <joint name="camera_joint" type="fixed">
         <axis xyz="0 1 0" />
-        <origin xyz="-0.1 0 .2" rpy="0 0 0"/>
+        <origin xyz="0.25 0.0 0.15" rpy="0 0 0"/>
         <parent link="base_link"/>
         <child link="camera_point_link"/>
@@ -214,5 +216,5 @@
 <!-- Gazebo references -->
   <gazebo reference="chassis">
-  	<material>Gazebo/Green</material>
+  	<material>Gazebo/DarkGrey</material>
     	<mu1>.01</mu1>
     	<mu2>.01</mu2>
@@ -222,5 +224,5 @@
   </gazebo>
   <gazebo reference="left_wheel">
-    	<material>Gazebo/Red</material>
+    	<material>Gazebo/FlatBlack</material>
     	<mu1>100000</mu1>
     	<mu2>100000</mu2>
@@ -230,5 +232,5 @@
   </gazebo>
   <gazebo reference="right_wheel">
-    	<material>Gazebo/Yellow</material>
+    	<material>Gazebo/FlatBlack</material>
     	<mu1>100000</mu1>
     	<mu2>100000</mu2>
@@ -238,5 +240,5 @@
   </gazebo>
   <gazebo reference="castor">
-  	<material>Gazebo/Blue</material>
+  	<material>Gazebo/FlatBlack</material>
     	<mu1>.01</mu1>
     	<mu2>.01</mu2>
